File: 010.Hardware/T12_SolderingStation.kicad_sch (KiCad schematic)
At the start: 51 parts

Commit message: 完成部分原理图
Parts:
- removed C?: 50V/100nF, Capacitor_SMD:C_0402_1005Metric, symbol Device:C
- added C? (x3): 4.7uF, Capacitor_SMD:C_0603_1608Metric, symbol Device:C
- added C? (x2): 100nF, symbol Device:C
- added C?: 50V/100nF, Capacitor_SMD:C_0402_1005Metric, symbol Device:C
- added C? (x2): 1uF, Capacitor_SMD:C_0603_1608Metric, symbol Device:C
- added C? (x2): 10uF, symbol Device:CP
- added C? (x2): 100nF, Capacitor_SMD:C_0603_1608Metric, symbol Device:C
- added C?: 2.2uF, Capacitor_SMD:C_0603_1608Metric, symbol Device:C
- added D?: 1N4148, Diode_SMD:D_SOD-123, symbol Device:D
- added J?: Conn_01x04_Male, symbol Connector:Conn_01x04_Male
- added R? (x2): 10K, symbol Device:R
- added R?: 100K, symbol Device:R
- added R?: 560K, Resistor_SMD:R_0402_1005Metric, symbol Device:R
- added RN?: 4.7K, Resistor_SMD:R_Array_Concave_4x0402, symbol Device:R_Pack04
- added U?: 0.91_OLED_128x32, Art_Pi_Sensor:OLED_128x32, symbol Art_Pi_Sensor-rescue:0.91_OLED_128x48
- added U?: RS0102YH8, Package_SO:VSSOP-8_2.3x2mm_P0.5mm, symbol My_Library:RS0102YH8
- added U?: RT9013-3V3, Package_TO_SOT_SMD:SOT-23-5, symbol Regulator_Linear:MIC5205-3.3YM5
Connections:
- net D10: now also J?.3 (Pin_3), R?.2
- net GND: now also J?.5 (Pin_5), C?.1, C?.2, C?.2, C?.2, C?.2, C?.2, C?.2, C?.2, C?.2, C?.2, C?.2, J?.4 (Pin_4), R?.2, U?.2 (GND), U?.5 (GND), U?.7 (VSS)
- net P+: now also J?.2 (Pin_2)
- net RST: now also RN?.4 (R4.1)
- net RXD: now also J?.3 (Pin_3)
- net SCL: now also U?.2 (B1)
- net SDA: now also U?.3 (B2)
- net TXD: now also J?.2 (Pin_2)
- net VBUS: now also J?.1 (Pin_1)
- net VCC: now also C?.1, C?.1, C?.1, J?.1 (Pin_1), R?.1, R?.1, R?.1, U?.1 (IN), U?.1 (VCCB)
- net ADC2: now reaches J?.4 (Pin_4)
- net ADC2: now also U?.25 (PC2)
- new net: C?.2, D?.2 (A), RN?.1 (R1.1), U?.9 (RES#)
- new net: C?.1, C?.1, U?.14 (VCC)
- new net: C?.1, U?.1 (C2P)
- new net: R?.1, U?.12 (IREF)
- new net: C?.1, U?.13 (VCOMH)
- new net: C?.2, U?.2 (C2N)
- new net: C?.1, U?.3 (C1P)
- new net: C?.2, U?.4 (C1N)
- new net: R?.2, U?.4 (OE)
- new net: R?.2, U?.3 (EN)
- new net +3V3: C?.1, C?.1, C?.1, C?.1, D?.1 (K), RN?.5 (R4.2), RN?.6 (R3.2), RN?.7 (R2.2), RN?.8 (R1.2), U?.5 (OUT), U?.5 (VBAT), U?.8 (VCCA), U?.8 (VDD)
- new net DISP_SCL: RN?.3 (R3.1), U?.10 (SCL), U?.7 (A1)
- new net DISP_SDA: RN?.2 (R2.1), U?.11 (SDA), U?.6 (A2)
Other:
- note added: "3V3_LDO"
- note added: "ATMEL328P"
- note added: "AVR_ISP"
- note added: "DC-DC"
- note added: "IIC_OLED"
- note added: "POWER_ADC&BEEP"
- note added: "ROTARY ENCODER"
- note added: "SOCKET"
- note added: "Thermocouple Amplifier"
- note added: "USB_PD_POWER"
- note added: "VL_TRANSLATOR"
- moved on the sheet: BZ?, C?, D?, J?, JP?, L?, Q?, R?, RV?, SW?, U?, U?A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

Commit message: 增加3D文件，完善原理图纸
Parts:
- removed SW?: RotaryEncoder_Switch, symbol Device:RotaryEncoder_Switch
- added C18: 100nF, Capacitor_SMD:C_0603_1608Metric, symbol Device:C
- added R21: 200K, Resistor_SMD:R_0402_1005Metric, symbol Device:R
- added SW1: SW_DPST_Temperature, Button_Switch_SMD:SW_SPST_Omron_B3FS-100xP, symbol Switch:SW_DPST_Temperature
- added SW2: RotaryEncoder_2, My_Library:EC10E, symbol My_Library:RotaryEncoder_2
- BZ1: renamed from BZ?; footprint (none) -> Buzzer_Beeper:Buzzer_12x9.5RM7.6
- C1, C3: renamed from C?; footprint Capacitor_SMD:C_0402_1005Metric -> Capacitor_SMD:C_0603_1608Metric
- C12, C13, C20, C26, C27, C5, C7: renamed from C?; footprint (none) -> Capacitor_SMD:C_0603_1608Metric
- C24, C4, C6: renamed from C?; footprint (none) -> Capacitor_SMD:C_1206_3216Metric
- C25: renamed from C?; value 2.2nF -> 100nF; footprint (none) -> Capacitor_SMD:C_0603_1608Metric
- J1: renamed from J?; footprint (none) -> Connector_USB:USB_C_Receptacle_Palconn_UTC16-G
- J3: renamed from J?; footprint (none) -> Connector_PinHeader_2.54mm:PinHeader_1x04_P2.54mm_Vertical
- J4: renamed from J?; footprint (none) -> Connector_Phoenix_MC:PhoenixContact_MC_1,5_5-G-3.5_1x05_P3.50mm_Horizontal
- Q1: renamed from Q?; footprint Package_TO_SOT_THT:TO-92_Inline -> Package_TO_SOT_SMD:TSOT-23
- R1, R10, R11, R14, R16, R17, R18, R19, R2, R20, R5, R9: renamed from R?; footprint (none) -> Resistor_SMD:R_0402_1005Metric
- R13: renamed from R?; value R -> 100K; footprint (none) -> Resistor_SMD:R_0402_1005Metric
- R15: renamed from R?; value R -> 20K; footprint (none) -> Resistor_SMD:R_0402_1005Metric
- U1: renamed from U?; footprint Package_SO:HSOP-8-1EP_3.9x4.9mm_P1.27mm_EP2.41x3.1mm -> Package_SO:SOIC-8-1EP_3.9x4.9mm_P1.27mm_EP2.29x3mm_ThermalVias
- U4: renamed from U?; footprint Art_Pi_Sensor:OLED_128x32 -> My_Library:OLED_128x32
- Y1: renamed from Y?; footprint (none) -> Crystal:Resonator_SMD_Murata_CSTxExxV-3Pin_3.0x1.1mm
- gave numbers to parts that had none: 35
Connections:
- net D6: now also SW1.2, SW1.4, SW2.B
- net D7: now also SW2.A
- net GND: now also C26.2, C27.2, D5.1 (K), U2.21 (GND), C18.2, R21.1, SW1.1, SW1.3, SW2.0 (SHELL), SW2.C; no longer U2.0 (GND)
- net at R20.1, U7.2 (-): now also R21.2
- net at U5.20 (AREF): now also C18.1
- no-connect marks 4 -> 8
Other:
- moved on the sheet: C20, R11
