File: 010.Hardware/T12_SolderingStationMain/T12_SolderingStation.kicad_sch (KiCad schematic)
At the start: 74 parts, among them J1 USB_C_Receptacle_USB2.0, J2 AVR-ISP-6, J3 Conn_01x04_Male, J4 Conn_01x05_Female, Q1 S8050, SW1 SW_DPST_Temperature, SW2 RotaryEncoder_2, U1 MP1584EN, U2 CH224D, U3 RT9013-3V3, U4 0.91_OLED_128x32, U5 ATmega328P-A, U6 RS0102YH8, U7 OPA2333xxD, Y1 16mHz

Commit message: 更新一点
Parts:
- removed BZ1: Buzzer, Buzzer_Beeper:Buzzer_12x9.5RM7.6, symbol Device:Buzzer
- removed C14, C15: 1uF, Capacitor_SMD:C_0603_1608Metric, symbol Device:C
- removed C16, C19, C22: 4.7uF, Capacitor_SMD:C_0603_1608Metric, symbol Device:C
- removed C17, C23, C5, C7: 100nF, Capacitor_SMD:C_0603_1608Metric, symbol Device:C
- removed C21: 2.2uF, Capacitor_SMD:C_0603_1608Metric, symbol Device:C
- removed C24: 10uF, Capacitor_SMD:C_1206_3216Metric, symbol Device:C_Polarized
- removed C4, C6: 10uF, Capacitor_SMD:C_1206_3216Metric, symbol Device:CP
- removed D3: 1N4148, Diode_SMD:D_SOD-123, symbol Device:D
- removed Q1: S8050, Package_TO_SOT_SMD:TSOT-23, symbol Transistor_BJT:S8050
- removed R12: 560K, Resistor_SMD:R_0402_1005Metric, symbol Device:R
- removed R14: 10K, Resistor_SMD:R_0402_1005Metric, symbol Device:R
- removed R5: 100K, Resistor_SMD:R_0402_1005Metric, symbol Device:R
- removed RN1: 4.7K, Resistor_SMD:R_Array_Concave_4x0402, symbol Device:R_Pack04
- removed RV1: 50K, Potentiometer_THT:Potentiometer_Bourns_3266W_Vertical, symbol Device:R_POT_Small
- removed U3: RT9013-3V3, Package_TO_SOT_SMD:SOT-23-5, symbol Regulator_Linear:MIC5205-3.3YM5
- removed U4: 0.91_OLED_128x32, My_Library:OLED_128x32, symbol Art_Pi_Sensor-rescue:0.91_OLED_128x48
- removed U6: RS0102YH8, Package_SO:VSSOP-8_2.3x2mm_P0.5mm, symbol My_Library:RS0102YH8
- added R4: 20K, Resistor_SMD:R_0402_1005Metric, symbol Device:R
- C8: renamed from C12; value 1uF -> 10uF; footprint Capacitor_SMD:C_0603_1608Metric -> Capacitor_SMD:C_0805_2012Metric
- D1: footprint Diode_SMD:D_SMB -> Diode_SMD:D_SMA
- renumbered C18 to C10, C20 to C11, C25 to C13, C26 to C14, C27 to C15, C8 to C4, C9 to C5, C10 to C6, C11 to C7, C13 to C9, D4 to D3, D5 to D4, R13 to R12, R15 to R13, R16 to R14, R17 to R15, R18 to R16, R19 to R17, R20 to R18, R21 to R19, R4 to R5, U5 to U3, U7 to U4
Connections:
- net VCC: now also R4.1
- net at R6.1, U1.4 (FB): now also R4.2
- no-connect marks 8 -> 6
Other:
- note removed: "3V3_LDO"
- note removed: "IIC_OLED"
- note removed: "VL_TRANSLATOR"
