File: 010.Hardware/T12_SolderingStationMain/T12_SolderingStation.kicad_sch (KiCad schematic)
At the start: 51 parts, among them J1 USB_C_Receptacle_USB2.0, J2 AVR-ISP-6, J3 Conn_01x04_Male, J4 Conn_01x05_Female, SW1 SW_DPST_Temperature, SW2 RotaryEncoder_2, U1 MP1584EN, U2 CH224D, U3 ATmega328P-A, U4 OPA2333xxD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

Commit message: 完善图纸
Parts:
- removed J2: AVR-ISP-6, Connector_PinHeader_2.54mm:PinHeader_2x03_P2.54mm_Vertical, symbol Connector:AVR-ISP-6
- removed J3: Conn_01x04_Male, Connector_PinHeader_2.54mm:PinHeader_1x04_P2.54mm_Vertical, symbol Connector:Conn_01x04_Male
- added D5: SDT10A45P5, My_Library:PowerDI5, symbol My_Library:SDT10A45P5
- added J5, J6: Conn_01x06_Female, Connector_PinHeader_2.54mm:PinHeader_1x06_P2.54mm_Vertical, symbol Connector:Conn_01x06_Female
- added TP1: VCC, TestPoint:TestPoint_Pad_1.0x1.0mm, symbol Connector:TestPoint
- added TP2: MISO, TestPoint:TestPoint_Pad_1.0x1.0mm, symbol Connector:TestPoint
- added TP3: MOSI, TestPoint:TestPoint_Pad_1.0x1.0mm, symbol Connector:TestPoint
- added TP4: SCK, TestPoint:TestPoint_Pad_1.0x1.0mm, symbol Connector:TestPoint
- added TP5: RST, TestPoint:TestPoint_Pad_1.0x1.0mm, symbol Connector:TestPoint
- added TP6: GND, TestPoint:TestPoint_Pad_1.0x1.0mm, symbol Connector:TestPoint
- added TP7: TXD, TestPoint:TestPoint_Pad_1.0x1.0mm, symbol Connector:TestPoint
- added TP8: RXD, TestPoint:TestPoint_Pad_1.0x1.0mm, symbol Connector:TestPoint
- C2: footprint Capacitor_SMD:CP_Elec_5x5.7 -> Capacitor_Tantalum_SMD:CP_EIA-3528-21_Kemet-B
- C4: footprint Capacitor_SMD:CP_Elec_5x5.7 -> Capacitor_Tantalum_SMD:CP_EIA-6032-28_Kemet-C
- JP1, JP2: footprint Jumper:SolderJumper-2_P1.3mm_Open_TrianglePad1.0x1.5mm -> Jumper:SolderJumper-2_P1.3mm_Open_RoundedPad1.0x1.5mm
Connections:
- net ADC2: now also J4.1 (Pin_1); no longer J4.4 (Pin_4)
- net BEEP: now also J5.6 (Pin_6)
- net D6: no longer SW2.B, U3.12 (PB0)
- net GND: now also J4.4 (Pin_4), J5.5 (Pin_5), J6.3 (Pin_3), J6.4 (Pin_4), TP6.1; no longer J4.5 (Pin_5)
- net MISO: now also TP2.1
- net MOSI: now also TP3.1
- net RST: now also J5.4 (Pin_4), TP5.1
- net RXD: now also TP8.1
- net SCK: now also TP4.1
- net SCL: now also J5.3 (Pin_3)
- net SDA: now also J5.2 (Pin_2)
- net TXD: now also TP7.1
- net VBUS: now also D5.1 (A), D5.2 (A); no longer C4.1, C5.1, J4.1 (Pin_1), R3.1, U1.7 (VIN)
- net VCC: now also J5.1 (Pin_1), TP1.1
- new net +24V: C4.1, C5.1, D5.3 (K), J4.5 (Pin_5), J6.1 (Pin_1), J6.2 (Pin_2), R3.1, U1.7 (VIN)
- new net D8: SW2.B, U3.12 (PB0)
- no-connect marks 6 -> 8
Other:
- moved on the sheet: J4, R14
