File: 010.Hardware/T12_SolderingStationScreen/T12_SolderingStationScreen.kicad_pcb (KiCad board)
At the start: 2 copper layers, 40 x 23 mm, 27 parts, among them J1 Conn_01x06_Female, J2 Conn_01x06_Female, Q1 S8050, U1 RT9013-3V3, U2 RS0102YH8, U3 0.91_OLED_128x32

Commit message: 完善图纸
Connections:
- C10 pad 2: Net-(C10-Pad2) -> /RST
- D1 pad 2: Net-(C10-Pad2) -> /RST
- J1 pad 4: unconnected-(J1-Pad4) -> /RST
- RN1 pad 1: Net-(C10-Pad2) -> unconnected-(RN1-Pad1)
- U3 pad 9: Net-(C10-Pad2) -> /RST
Routing:
- net +3V3: track 0.00 -> 12.5 mm, vias 0 -> 1
- net GND: track 0.00 -> 8.54 mm
- net /RST: track 0.00 -> 7.86 mm
- net /DISP_SDA: track 0.00 -> 7.27 mm
- net /DISP_SCL: track 0.00 -> 6.97 mm
- net Net-(C5-Pad1): track 0.00 -> 5.81 mm, vias 0 -> 1
- net Net-(C6-Pad1): track 0.00 -> 5.15 mm, vias 0 -> 1
- net Net-(C11-Pad1): track 0.00 -> 5.05 mm, vias 0 -> 1
- net Net-(R4-Pad1): track 0.00 -> 4.90 mm
- net Net-(C12-Pad1): track 0.00 -> 4.49 mm, vias 0 -> 1
- net Net-(C6-Pad2): track 0.00 -> 3.44 mm, vias 0 -> 1
- net Net-(C5-Pad2): track 0.00 -> 3.03 mm, vias 0 -> 1

Commit message: 完善图纸
Parts:
- moved JP1 7.22 mm to (102.4, 128.8), turned to 0 degrees
- moved R2 2.79 mm to (113.3, 127.3), turned to 90 degrees
- moved Q1 0.08 mm to (112.6, 120.4)
- turned C3 to 180 degrees
Routing:
- net GND: track 8.54 -> 71.3 mm, vias 0 -> 131
- net VCC: track 0.00 -> 43.7 mm, vias 0 -> 3
- net Net-(Q1-Pad2): track 0.00 -> 24.0 mm
- net /RST: track 7.86 -> 26.8 mm, vias 0 -> 1
- net +3V3: track 12.5 -> 27.4 mm
- net /SCL: track 0.00 -> 10.5 mm
- net /SDA: track 0.00 -> 8.89 mm
- net Net-(BZ1-Pad2): track 0.00 -> 6.70 mm
- net Net-(C3-Pad1): track 0.00 -> 5.88 mm
- net /BEEP: track 0.00 -> 2.96 mm
- net +24V: track 0.00 -> 2.54 mm
- net Net-(C5-Pad1): track 5.81 -> 3.27 mm
- net Net-(R2-Pad2): track 0.00 -> 2.49 mm
- net Net-(C5-Pad2): track 3.03 -> 5.02 mm
- net Net-(C6-Pad1): track 5.15 -> 3.38 mm
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- added copper zone on B.Cu, net GND
- added copper zone on F.Cu, net GND
