File: 010.Hardware/T12_SolderingStationScreen/T12_SolderingStationScreen.kicad_sch (KiCad schematic)
At the start: 23 parts

Commit message: 完善图纸
Parts:
- removed C? (x2): 10uF, Capacitor_SMD:C_1206_3216Metric, symbol Device:CP
- added C1: 10uF, Capacitor_Tantalum_SMD:CP_EIA-6032-28_Kemet-C, symbol Device:C_Polarized
- added C3: 10uF, Capacitor_Tantalum_SMD:CP_EIA-3528-21_Kemet-B, symbol Device:C_Polarized
- added J1, J2: Conn_01x06_Female, Connector_PinSocket_2.54mm:PinSocket_1x06_P2.54mm_Vertical, symbol Connector:Conn_01x06_Female
- added JP1: JUMP, Jumper:SolderJumper-2_P1.3mm_Bridged2Bar_Pad1.0x1.5mm, symbol Jumper:SolderJumper_2_Bridged
- added R3: 2K, Resistor_SMD:R_0402_1005Metric, symbol Device:R
- gave numbers to parts that had none: 21
Connections:
- net +3V3: now also JP1.1 (A); no longer C4.1, U1.5 (OUT)
- net BEEP: now also J1.6 (Pin_6), R3.2
- net GND: now also C1.2, C3.2, J1.5 (Pin_5), J2.3 (Pin_3), J2.4 (Pin_4)
- net SCL: now also J1.3 (Pin_3)
- net SDA: now also J1.2 (Pin_2)
- net VCC: now also C1.1, J1.1 (Pin_1)
- net at Q1.2 (B): now also R3.1
- new net: C3.1, C4.1, JP1.2 (B), U1.5 (OUT)
- new net +24V: J2.1 (Pin_1), J2.2 (Pin_2)
- no-connect marks 2 -> 5
Other:
- moved on the sheet: BZ1, C10, C11, C12, C13, C5, C6, C7, C8, C9, D1, Q1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

Commit message: 完善图纸
Connections:
- net RST: now also C10.2, D1.2 (A), J1.4 (Pin_4), U3.9 (RES#)
- now unconnected: RN1.1 (R1.1)
- no-connect marks 5 -> 4
Changed lines of the file:
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@@
   (junction (at 67.31 83.82) (diameter 0) (color 0 0 0 0)
   )
-  (junction (at 41.91 93.98) (diameter 0) (color 0 0 0 0)
-  )
   (junction (at 44.45 82.55) (diameter 0) (color 0 0 0 0)
   )
+  (junction (at 49.53 93.98) (diameter 0) (color 0 0 0 0)
+  )
   (junction (at 46.99 82.55) (diameter 0) (color 0 0 0 0)
   )
@@
   )
   (no_connect (at 76.2 86.36))
-  (no_connect (at 161.29 127))
   (no_connect (at 69.85 39.37))
   (no_connect (at 190.5 132.08))
@@
     (stroke (width 0) (type default) (color 0 0 0 0))
   )
-  (wire (pts (xy 49.53 92.71) (xy 55.88 92.71))
-    (stroke (width 0) (type default) (color 0 0 0 0))
-  )
   (wire (pts (xy 199.39 102.87) (xy 199.39 100.33))
     (stroke (width 0) (type default) (color 0 0 0 0))
@@
     (stroke (width 0) (type default) (color 0 0 0 0))
   )
-  (wire (pts (xy 41.91 92.71) (xy 41.91 93.98))
-    (stroke (width 0) (type default) (color 0 0 0 0))
-  )
   (wire (pts (xy 190.5 121.92) (xy 198.12 121.92))
     (stroke (width 0) (type default) (color 0 0 0 0))
@@
     (stroke (width 0) (type default) (color 0 0 0 0))
   )
-  (wire (pts (xy 41.91 93.98) (xy 76.2 93.98))
+  (wire (pts (xy 36.83 93.98) (xy 49.53 93.98))
     (stroke (width 0) (type default) (color 0 0 0 0))
   )
@@
     (stroke (width 0) (type default) (color 0 0 0 0))
   )
-  (wire (pts (xy 36.83 93.98) (xy 41.91 93.98))
-    (stroke (width 0) (type default) (color 0 0 0 0))
-  )
   (wire (pts (xy 198.12 119.38) (xy 201.93 119.38))
     (stroke (width 0) (type default) (color 0 0 0 0))
@@
     (stroke (width 0) (type default) (color 0 0 0 0))
   )
+  (wire (pts (xy 49.53 93.98) (xy 49.53 92.71))
+    (stroke (width 0) (type default) (color 0 0 0 0))
+  )
   (wire (pts (xy 36.83 82.55) (xy 41.91 82.55))
     (stroke (width 0) (type default) (color 0 0 0 0))
@@
   )
   (wire (pts (xy 52.07 39.37) (xy 52.07 43.18))
+    (stroke (width 0) (type default) (color 0 0 0 0))
+  )
+  (wire (pts (xy 49.53 93.98) (xy 76.2 93.98))
     (stroke (width 0) (type default) (color 0 0 0 0))
   )
@@
     (effects (font (size 2.54 2.54) (thickness 0.508) bold) (justify left bottom))
   )
+  (label "RST" (at 67.31 93.98 0)
+    (effects (font (size 1.27 1.27)) (justify left bottom))
+  )
   (label "SCL" (at 148.59 124.46 0)
     (effects (font (size 1.27 1.27)) (justify left bottom))
   )
+  (label "RST" (at 148.59 127 0)
+    (effects (font (size 1.27 1.27)) (justify left bottom))
+  )
   (label "DISP_SCL" (at 207.01 41.91 0)
     (effects (font (size 1.27 1.27)) (justify left bottom))
@@
   )
   (label "BEEP" (at 170.18 92.71 0)
-    (effects (font (size 1.27 1.27)) (justify left bottom))
-  )
-  (label "RST" (at 52.07 92.71 0)
     (effects (font (size 1.27 1.27)) (justify left bottom))
   )
@@
   (symbol (lib_id "Device:C") (at 63.5 91.44 270) (unit 1)
     (in_bom yes) (on_board yes)
-    (property "Reference" "C9" (id 0) (at 59.69 92.71 90)
-      (effects (font (size 1.27 1.27)) (justify left))
-    )
-    (property "Value" "100nF" (id 1) (at 64.77 92.71 90)
-      (effects (font (size 1.27 1.27)) (justify left))
-    )
+    (property "Reference" "C9" (id 0) (at 59.69 90.17 90)
+      (effects (font (size 1.27 1.27)) (justify left))
+    )
+    (property "Value" "100nF" (id 1) (at 57.15 92.71 90)
+      (effects (font (size 1.27 1.27)) (justify left))
+    )
